File: 40_Implementation/10_HW/XX_PCB_template/10_work/80_KiCad/80_KiCad.kicad_pcb (KiCad board)
At the start: 4 copper layers, 68.6 x 53.3 mm, 42 parts, among them J1 Power, J2 Digital/PWM, J3 Analog, J4 Digital/PWM, J5 Conn_01x03_Socket, SW1 SW_SPST, U1 OPA340P, U2 OPA340P

Commit message: Almost Submitted
Parts:
- moved A1_In_N 1.28 mm to (102.7, 66.6)
- moved A_In_P 1.15 mm to (102.8, 89.5)
- moved J5 0.40 mm to (158.0, 73.9)
Other:
- board text added: "Movement Detector Group D3 Rakshita (1127990) Zaki (1127995)"
- board text removed: "Movement Detector Rakshita (1127990) Zaki (1127995) ${REVISION}"
Changed lines of the file:
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@@
 		(title "Movement Detector")
 		(date "2024-05-05")
-		(rev "v1.1")
+		(rev "v1.0")
 		(company "Hochschule Darmstadt")
 	)
@@
 		(tags "LED diameter 5.0mm 2 pins")
 		(property "Reference" "D2"
-			(at 1.27 -3.96 0)
+			(at -2.225 -3 0)
 			(layer "F.SilkS")
 			(effects
@@
 		(tags "LED diameter 5.0mm 2 pins")
 		(property "Reference" "D3"
-			(at 1.27 -3.96 0)
+			(at -2.4 -3.175 0)
 			(layer "F.SilkS")
 			(effects
@@
 	(footprint "Connector_PinHeader_2.54mm:PinHeader_1x01_P2.54mm_Vertical"
 		(layer "F.Cu")
-		(at 102.825 88.325)
+		(at 102.775 89.475)
 		(descr "Through hole straight pin header, 1x01, 2.54mm pitch, single row")
 		(tags "Through hole pin header THT 1x01 2.54mm single row")
 		(property "Reference" "A_In_P"
-			(at 2.75 -0.725 270)
+			(at 0.275 -2.525 0)
 			(layer "F.SilkS")
 			(effects
@@
 	(footprint "Connector_PinHeader_2.54mm:PinHeader_1x01_P2.54mm_Vertical"
 		(layer "F.Cu")
-		(at 102.725 65.35)
+		(at 102.65 66.625)
 		(descr "Through hole straight pin header, 1x01, 2.54mm pitch, single row")
 		(tags "Through hole pin header THT 1x01 2.54mm single row")
 		(property "Reference" "A1_In_N"
-			(at 2.25 0.175 270)
+			(at 0.55 -2.575 0)
 			(layer "F.SilkS")
 			(effects
@@
 		(tags "C Rect series Radial pin pitch 5.00mm  length 7.2mm width 7.2mm Capacitor")
 		(property "Reference" "C5"
-			(at 2.675 -4.5 0)
+			(at 8.025 -0.225 0)
 			(layer "F.SilkS")
 			(effects
@@
 		(tags "Resistor Axial_DIN0207 series Axial Horizontal pin pitch 10.16mm 0.25W = 1/4W length 6.3mm diameter 2.5mm")
 		(property "Reference" "R5"
-			(at 5.08 -2.37 90)
+			(at 4.83 -2.525 180)
 			(layer "F.SilkS")
 			(effects
@@
 		(tags "LED diameter 5.0mm 2 pins")
 		(property "Reference" "D1"
-			(at 1.375 -4.25 180)
+			(at -2.85 -3.025 180)
 			(layer "F.SilkS")
 			(effects
@@
 		(tags "C Rect series Radial pin pitch 5.00mm  length 7.2mm width 2.5mm Capacitor")
 		(property "Reference" "C1"
-			(at 2.5 -2.5 -90)
+			(at 3.175 -2.775 0)
 			(layer "F.SilkS")
 			(effects
@@
 		(tags "Through hole pin header THT 1x01 2.54mm single row")
 		(property "Reference" "A1_Out"
-			(at 0.775 -3.55 0)
+			(at 0.625 -3.025 0)
 			(layer "F.SilkS")
 			(effects
@@
 		(tags "C Rect series Radial pin pitch 5.00mm  length 7.2mm width 7.2mm Capacitor")
 		(property "Reference" "C6"
-			(at 2.5 -4.85 180)
+			(at -2.725 0.3 180)
 			(layer "F.SilkS")
 			(effects
@@
 	(footprint "Connector_PinSocket_2.54mm:PinSocket_1x03_P2.54mm_Horizontal"
 		(layer "F.Cu")
-		(at 157.625 73.85 180)
+		(at 158.025 73.875 180)
 		(descr "Through hole angled socket strip, 1x03, 2.54mm pitch, 8.51mm socket length, single row (from Kicad 4.0.7), script generated")
 		(tags "Through hole angled socket strip THT 1x03 2.54mm single row")
@@
 		(layer "Edge.Cuts")
 	)
-	(gr_text "Movement Detector\nRakshita (1127990)\nZaki (1127995)\n${REVISION}"
-		(at 115.85 91.975 90)
+	(gr_text "Movement Detector\nGroup D3\nRakshita (1127990)\nZaki (1127995)"
+		(at 105.65 85.65 0)
 		(layer "F.SilkS")
 		(effects
 			(font
-				(size 1 1)
+				(size 0.8 0.8)
 				(thickness 0.15)
 			)
@@
 	)
 	(segment
-		(start 105.025 90.525)
-		(end 102.825 88.325)
+		(start 103.975 89.475)
+		(end 102.775 89.475)
 		(width 0.25)
 		(layer "F.Cu")
@@
 	)
 	(segment
+		(start 105.025 90.525)
+		(end 103.975 89.475)
+		(width 0.25)
+		(layer "F.Cu")
+		(net 31)
+	)
+	(segment
 		(start 129.82 88.975)
 		(end 130.05 89.205)
@@
 	)
 	(segment
-		(start 157.625 71.31)
-		(end 154.529888 71.31)
-		(width 0.25)
-		(layer "F.Cu")
-		(net 32)
-	)
-	(segment
 		(start 156.7 92.75)
 		(end 156.7 91.075)
@@
 	)
 	(segment
-		(start 154.529888 71.31)
+		(start 154.554888 71.335)
 		(end 153.869888 70.65)
 		(width 0.25)
@@
 	)
 	(segment
+		(start 158.025 71.335)
+		(end 154.554888 71.335)
+		(width 0.25)
+		(layer "F.Cu")
+		(net 32)
+	)
+	(segment
 		(start 154.1 70.880112)
 		(end 153.869888 70.65)
@@
 	)
 	(segment
-		(start 105.6 68.225)
-		(end 102.725 65.35)
+		(start 104.325 68.3)
+		(end 102.65 66.625)
 		(width 0.25)
 		(layer "F.Cu")
@@
 	)
 	(segment
-		(start 131.2 77.975)
-		(end 133.225 75.95)
+		(start 130.225 65.94)
+		(end 127.865 68.3)
 		(width 0.25)
 		(layer "F.Cu")
@@
 	)
 	(segment
-		(start 135.34 60.825)
-		(end 130.225 65.94)
+		(start 131.2 77.975)
+		(end 133.225 75.95)
 		(width 0.25)
 		(layer "F.Cu")
@@
 	)
 	(segment
-		(start 130.225 65.94)
-		(end 127.94 68.225)
+		(start 135.34 60.825)
+		(end 130.225 65.94)
 		(width 0.25)
 		(layer "F.Cu")
@@
 	)
 	(segment
-		(start 127.94 68.225)
-		(end 105.6 68.225)
+		(start 127.865 68.3)
+		(end 104.325 68.3)
 		(width 0.25)
 		(layer "F.Cu")
@@
 			(clearance 0.508)
 		)
-		(min_thickness 0.4)
+		(min_thickness 0.25)
 		(filled_areas_thickness no)
 		(fill yes
@@
 			(clearance 0.508)
 		)
-		(min_thickness 0.4)
+		(min_thickness 0.25)
 		(filled_areas_thickness no)
 		(fill yes
@@
 			(clearance 0.508)
 		)
-		(min_thickness 0.4)
+		(min_thickness 0.25)
 		(filled_areas_thickness no)
 		(fill yes
@@
 			(clearance 0.508)
 		)
-		(min_thickness 0.4)
+		(min_thickness 0.25)
 		(filled_areas_thickness no)
 		(fill yes
